File: sensor/sensor.kicad_pcb (KiCad board)
At the start: 2 copper layers, 19.6 x 13.2 mm, 4 parts, among them J2 Conn_01x03, U1 KMZ60

Commit message: kicad
Parts:
- REF** (x2): value MountingHole_2.2mm_M2 -> (none)
Routing:
- net (no net): track 24.0 -> 0.00 mm
Other:
- net class Default: clearance 0.45 -> 0.8; trace_width 0.5 -> 0.45
- rule trace_clearance: 0.45 -> 0.8
Changed lines of the file:
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@@
-(kicad_pcb (version 4) (host pcbnew 4.0.7)
+(kicad_pcb (version 4) (host pcbnew 4.0.7-e2-6376~58~ubuntu16.04.1)
   (general
     (links 4)
     (no_connects 0)
-    (area 140.640999 103.865 160.349001 121.329619)
+    (area 139.726999 103.515 161.263001 121.679619)
     (thickness 1.6)
     (drawings 11)
-    (tracks 35)
+    (tracks 19)
     (zones 0)
     (modules 4)
@@
   )
   (setup
-    (last_trace_width 0.5)
-    (trace_clearance 0.45)
+    (last_trace_width 0.45)
+    (trace_clearance 0.8)
     (zone_clearance 0.508)
     (zone_45_only no)
@@
     (mod_text_size 1 1)
     (mod_text_width 0.15)
-    (pad_size 1.7 1.7)
-    (pad_drill 1)
+    (pad_size 1.75 0.46)
+    (pad_drill 0)
     (pad_to_mask_clearance 0.2)
     (aux_axis_origin 143.002 108.331)
@@
   (net 7 "Net-(J1-Pad8)")
   (net_class Default "This is the default net class."
-    (clearance 0.45)
-    (trace_width 0.5)
+    (clearance 0.8)
+    (trace_width 0.45)
     (via_dia 0.6)
     (via_drill 0.4)
@@
     (fp_line (start -2.75 3.205) (end 2.75 3.205) (layer F.SilkS) (width 0.15))
     (fp_line (start -2.75 -2.55) (end -4.5 -2.55) (layer F.SilkS) (width 0.15))
-    (pad 1 smd rect (at -3.7 -1.905) (size 1.75 0.55) (layers F.Cu F.Paste F.Mask)
+    (pad 1 smd rect (at -3.7 -1.905) (size 1.75 0.46) (layers F.Cu F.Paste F.Mask)
       (net 1 "Net-(J1-Pad1)"))
-    (pad 2 smd rect (at -3.7 -0.635) (size 1.75 0.55) (layers F.Cu F.Paste F.Mask)
+    (pad 2 smd rect (at -3.7 -0.635) (size 1.75 0.46) (layers F.Cu F.Paste F.Mask)
       (net 2 "Net-(J1-Pad2)"))
-    (pad 3 smd rect (at -3.7 0.635) (size 1.75 0.55) (layers F.Cu F.Paste F.Mask)
+    (pad 3 smd rect (at -3.7 0.635) (size 1.75 0.46) (layers F.Cu F.Paste F.Mask)
       (net 3 "Net-(J1-Pad3)"))
-    (pad 4 smd rect (at -3.7 1.905) (size 1.75 0.55) (layers F.Cu F.Paste F.Mask)
+    (pad 4 smd rect (at -3.7 1.905) (size 1.75 0.46) (layers F.Cu F.Paste F.Mask)
       (net 4 "Net-(J1-Pad4)"))
-    (pad 5 smd rect (at 3.7 1.905) (size 1.75 0.55) (layers F.Cu F.Paste F.Mask)
+    (pad 5 smd rect (at 3.7 1.905) (size 1.75 0.46) (layers F.Cu F.Paste F.Mask)
       (net 5 "Net-(J1-Pad5)"))
-    (pad 6 smd rect (at 3.7 0.635) (size 1.75 0.55) (layers F.Cu F.Paste F.Mask)
+    (pad 6 smd rect (at 3.7 0.635) (size 1.75 0.46) (layers F.Cu F.Paste F.Mask)
       (net 6 "Net-(J1-Pad6)"))
-    (pad 7 smd rect (at 3.7 -0.635) (size 1.75 0.55) (layers F.Cu F.Paste F.Mask)
+    (pad 7 smd rect (at 3.7 -0.635) (size 1.75 0.46) (layers F.Cu F.Paste F.Mask)
       (net 1 "Net-(J1-Pad1)"))
-    (pad 8 smd rect (at 3.7 -1.905) (size 1.75 0.55) (layers F.Cu F.Paste F.Mask)
+    (pad 8 smd rect (at 3.7 -1.905) (size 1.75 0.46) (layers F.Cu F.Paste F.Mask)
       (net 7 "Net-(J1-Pad8)"))
     (model ${KISYS3DMOD}/Housings_SOIC.3dshapes/SO-8_5.3x6.2mm_Pitch1.27mm.wrl
@@
       (effects (font (size 1 1) (thickness 0.15)))
     )
-    (fp_text value MountingHole_2.2mm_M2 (at 0 3.2) (layer F.Fab)
+    (fp_text value "" (at 0 3.2) (layer F.Fab)
       (effects (font (size 1 1) (thickness 0.15)))
     )
@@
       (effects (font (size 1 1) (thickness 0.15)))
     )
-    (fp_text value MountingHole_2.2mm_M2 (at 0 3.2) (layer F.Fab)
+    (fp_text value "" (at 0 3.2) (layer F.Fab)
       (effects (font (size 1 1) (thickness 0.15)))
     )
@@
   (gr_line (start 140.716 107.188) (end 142.748 105.156) (angle 90) (layer Edge.Cuts) (width 0.15))
   (gr_line (start 140.716 108.204) (end 140.716 107.188) (angle 90) (layer Edge.Cuts) (width 0.15))
-  (segment (start 157.353 110.363) (end 159.004 110.363) (width 0.5) (layer F.Cu) (net 0))
-  (segment (start 159.004 110.363) (end 159.258 110.109) (width 0.5) (layer F.Cu) (net 0))
-  (segment (start 142.24 110.109) (end 142.24 112.268) (width 0.5) (layer F.Cu) (net 0))
-  (segment (start 143.256 110.998) (end 143.256 113.538) (width 0.5) (layer F.Cu) (net 0))
-  (segment (start 143.256 113.538) (end 144.5895 114.8715) (width 0.5) (layer F.Cu) (net 0))
-  (segment (start 157.1625 111.8235) (end 157.607 111.379) (width 0.5) (layer F.Cu) (net 0))
-  (segment (start 157.607 111.379) (end 159.004 111.379) (width 0.5) (layer F.Cu) (net 0))
-  (segment (start 156.1465 114.4905) (end 158.242 112.395) (width 0.5) (layer F.Cu) (net 0))
-  (segment (start 158.623 112.395) (end 159.131 112.903) (width 0.5) (layer F.Cu) (net 0))
-  (segment (start 158.242 112.395) (end 158.623 112.395) (width 0.5) (layer F.Cu) (net 0))
-  (segment (start 156.21 110.871) (end 156.21 112.776) (width 0.5) (layer F.Cu) (net 0))
-  (segment (start 156.21 112.776) (end 155.067 113.919) (width 0.5) (layer F.Cu) (net 0))
-  (segment (start 145.034 108.458) (end 145.034 109.601) (width 0.5) (layer F.Cu) (net 0))
-  (segment (start 144.272 112.903) (end 145.034 113.665) (width 0.5) (layer F.Cu) (net 0))
-  (segment (start 144.272 110.363) (end 144.272 112.903) (width 0.5) (layer F.Cu) (net 0))
-  (segment (start 145.034 109.601) (end 144.272 110.363) (width 0.5) (layer F.Cu) (net 0))
-  (segment (start 146.795 107.315) (end 145.288 107.315) (width 0.5) (layer F.Cu) (net 1))
-  (segment (start 149.479 105.918) (end 152.146 108.585) (width 0.5) (layer F.Cu) (net 1))
-  (segment (start 145.288 105.918) (end 149.479 105.918) (width 0.5) (layer F.Cu) (net 1))
-  (segment (start 145.034 106.172) (end 145.288 105.918) (width 0.5) (layer F.Cu) (net 1))
-  (segment (start 145.034 107.061) (end 145.034 106.172) (width 0.5) (layer F.Cu) (net 1))
-  (segment (start 145.288 107.315) (end 145.034 107.061) (width 0.5) (layer F.Cu) (net 1))
+  (segment (start 146.795 107.315) (end 145.288 107.315) (width 0.45) (layer F.Cu) (net 1))
+  (segment (start 149.479 105.918) (end 152.146 108.585) (width 0.45) (layer F.Cu) (net 1))
+  (segment (start 145.288 105.918) (end 149.479 105.918) (width 0.45) (layer F.Cu) (net 1))
+  (segment (start 145.034 106.172) (end 145.288 105.918) (width 0.45) (layer F.Cu) (net 1))
+  (segment (start 145.034 107.061) (end 145.034 106.172) (width 0.45) (layer F.Cu) (net 1))
+  (segment (start 145.288 107.315) (end 145.034 107.061) (width 0.45) (layer F.Cu) (net 1))
   (segment (start 154.195 108.585) (end 152.146 108.585) (width 0.5) (layer F.Cu) (net 1))
-  (segment (start 150.622 110.109) (end 150.622 116.332) (width 0.5) (layer F.Cu) (net 1))
-  (segment (start 152.146 108.585) (end 150.622 110.109) (width 0.5) (layer F.Cu) (net 1))
-  (segment (start 146.795 108.585) (end 148.463 108.585) (width 0.5) (layer F.Cu) (net 2))
-  (segment (start 148.082 114.046) (end 148.082 116.332) (width 0.5) (layer F.Cu) (net 2))
-  (segment (start 149.225 112.903) (end 148.082 114.046) (width 0.5) (layer F.Cu) (net 2))
-  (segment (start 149.225 109.347) (end 149.225 112.903) (width 0.5) (layer F.Cu) (net 2))
-  (segment (start 148.463 108.585) (end 149.225 109.347) (width 0.5) (layer F.Cu) (net 2))
+  (segment (start 150.622 110.109) (end 150.622 116.332) (width 0.45) (layer F.Cu) (net 1))
+  (segment (start 152.146 108.585) (end 150.622 110.109) (width 0.45) (layer F.Cu) (net 1))
+  (segment (start 146.795 108.585) (end 148.463 108.585) (width 0.45) (layer F.Cu) (net 2))
+  (segment (start 148.463 108.585) (end 149.225 109.347) (width 0.45) (layer F.Cu) (net 2))
+  (segment (start 149.225 109.347) (end 149.225 112.903) (width 0.45) (layer F.Cu) (net 2))
+  (segment (start 149.225 112.903) (end 148.082 114.046) (width 0.45) (layer F.Cu) (net 2))
+  (segment (start 148.082 114.046) (end 148.082 116.332) (width 0.45) (layer F.Cu) (net 2))
   (segment (start 154.195 109.855) (end 152.654 109.855) (width 0.5) (layer F.Cu) (net 6))
   (segment (start 153.162 114.173) (end 153.162 116.332) (width 0.5) (layer F.Cu) (net 6))
