File: kicad/starfish.kicad_pcb (KiCad board)
At the start: 2 copper layers, 3 parts, among them J1 Conn_02x04_Counter_Clockwise, J2 Conn_01x04, U1 kmz60

Commit message: kicad
Parts:
- removed U1: kmz60, Housings_SOIC:SO-8_5.3x6.2mm_Pitch1.27mm
- added J3: Conn_01x08, Pin_Headers:Pin_Header_Straight_1x08_Pitch2.54mm, F.Cu at (166.4, 118.1)
- added J4: Conn_01x08, Pin_Headers:Pin_Header_Straight_1x08_Pitch2.54mm, F.Cu at (166.4, 144.8)
- added J5: Conn_02x03_Counter_Clockwise, Pin_Headers:Pin_Header_Straight_2x03_Pitch2.54mm, F.Cu at (127.0, 95.2)
- added J6: Conn_01x05, Pin_Headers:Pin_Header_Straight_1x05_Pitch2.54mm, F.Cu at (185.4, 123.2)
- J1: value Conn_02x04_Counter_Clockwise -> Conn_01x09; footprint Pin_Headers:Pin_Header_Straight_2x04_Pitch2.54mm -> Pin_Headers:Pin_Header_Straight_1x09_Pitch2.54mm
- J2: value Conn_01x04 -> Conn_02x03_Counter_Clockwise; footprint Pin_Headers:Pin_Header_Straight_1x04_Pitch2.54mm -> Pin_Headers:Pin_Header_Straight_2x03_Pitch2.54mm
- moved J1 41.5 mm to (125.7, 132.1), turned to 180 degrees
- moved J2 35.9 mm to (170.2, 90.2), turned to 0 degrees
Connections:
- J1 pad 6: Net-(J1-Pad3) -> Net-(J1-Pad6)
- J2 pad 1: Net-(J1-Pad2) -> Net-(J2-Pad1)
- J2 pad 2: Net-(J1-Pad7) -> Net-(J1-Pad1)
- J2 pad 3: Net-(J1-Pad4) -> Net-(J2-Pad3)

Commit message: kicad
Parts:
- J1: value Conn_01x09 -> (none)
- J2: value Conn_02x03_Counter_Clockwise -> Sensor R
- J3: value Conn_01x08 -> MPU
- J4: value Conn_01x08 -> (none)
- J5: value Conn_02x03_Counter_Clockwise -> Sensor L
- J6: value Conn_01x05 -> (none)
- moved J2 28.6 mm to (147.8, 108.0)
- moved J6 21.6 mm to (164.0, 126.3)
- moved J3 16.9 mm to (150.4, 123.4)
- moved J5 13.9 mm to (132.6, 108.0)
- moved J1 8.53 mm to (118.9, 137.2)
- moved J4 8.02 mm to (159.2, 141.3)
Connections:
- J6 pad 1: Net-(J3-Pad5) -> Net-(J6-Pad1)
- J6 pad 2: Net-(J3-Pad6) -> Net-(J3-Pad5)
- J6 pad 3: Net-(J6-Pad3) -> Net-(J3-Pad6)
- J6 pad 5: Net-(J1-Pad3) -> Net-(J6-Pad5)
Routing:
- net Net-(J1-Pad3): track 0.00 -> 99.2 mm, vias 0 -> 5
- net Net-(J4-Pad2): track 0.00 -> 66.5 mm, vias 0 -> 1
- net Net-(J1-Pad1): track 0.00 -> 56.4 mm, vias 0 -> 1
- net Net-(J2-Pad6): track 0.00 -> 39.2 mm, vias 0 -> 1
- net Net-(J3-Pad6): track 0.00 -> 29.7 mm, vias 0 -> 1
- net Net-(J3-Pad5): track 0.00 -> 26.1 mm, vias 0 -> 1
- added copper zone on B.Cu, net Net-(J1-Pad3)
- added copper zone on F.Cu, net Net-(J1-Pad3)
Other:
- board outline added: 50 x 38.4 mm
- net class Default: clearance 0.2 -> 0.79375; trace_width 0.25 -> 0.35; via_dia 0.6 -> 1.2; via_drill 0.4 -> 0.79375
- rule trace_clearance: 0.2 -> 0.79375

Commit message: kicad
Other:
- net class Default: clearance 0.79375 -> 0.8
- rule trace_clearance: 0.79375 -> 0.8
Changed lines of the file:
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@@
   (page A4)
   (layers
-    (0 F.Cu signal hide)
+    (0 F.Cu signal)
     (31 B.Cu signal)
     (32 B.Adhes user)
@@
   (setup
     (last_trace_width 0.35)
-    (trace_clearance 0.79375)
+    (trace_clearance 0.8)
     (zone_clearance 0.508)
     (zone_45_only no)
@@
   (net 31 "Net-(J6-Pad5)")
   (net_class Default "This is the default net class."
-    (clearance 0.79375)
+    (clearance 0.8)
     (trace_width 0.35)
     (via_dia 1.2)
@@
   (segment (start 135.1153 129.2733) (end 135.0518 129.3368) (width 0.35) (layer B.Cu) (net 3))
   (via (at 135.0518 129.3368) (size 1.2) (drill 0.79375) (layers F.Cu B.Cu) (net 3))
-  (segment (start 154.08656 139.30376) (end 154.08656 141.25956) (width 0.35) (layer F.Cu) (net 3) (status 800000))
+  (segment (start 154.08656 139.30376) (end 154.08656 141.25956) (width 0.35) (layer F.Cu) (net 3))
   (segment (start 147.2692 132.4864) (end 154.08656 139.30376) (width 0.35) (layer F.Cu) (net 3))
   (segment (start 143.7132 132.4864) (end 147.2692 132.4864) (width 0.35) (layer F.Cu) (net 3))
@@
   (segment (start 132.1054 133.8326) (end 152.8572 133.8326) (width 0.35) (layer B.Cu) (net 20))
   (segment (start 152.86736 133.84276) (end 156.5656 137.5156) (width 0.35) (layer F.Cu) (net 20))
-  (segment (start 156.5656 137.5156) (end 156.62656 141.25956) (width 0.35) (layer F.Cu) (net 20) (status 800000))
+  (segment (start 156.5656 137.5156) (end 156.62656 141.25956) (width 0.35) (layer F.Cu) (net 20))
   (via (at 152.8572 133.8326) (size 1.2) (drill 0.79375) (layers F.Cu B.Cu) (net 20))
   (segment (start 152.86736 133.84276) (end 152.8572 133.8326) (width 0.35) (layer F.Cu) (net 20))

Commit message: shield
Parts:
- J1: value (none) -> Conn_01x09
- J2: value Sensor R -> conn1
- J3: value MPU -> Conn_01x08
- J4: value (none) -> Conn_01x08
- J5: value Sensor L -> conn2
- J6: value (none) -> Conn_01x05
- moved J5 16.0 mm to (148.6, 108.5)
- moved J2 15.0 mm to (132.8, 108.5)
Connections:
- J2 pad 2: Net-(J1-Pad1) -> Net-(J2-Pad2)
- J2 pad 3: Net-(J2-Pad3) -> Net-(J1-Pad1)
- J2 pad 5: Net-(J2-Pad5) -> Net-(J1-Pad2)
- J4 pad 1: Net-(J2-Pad6) -> Net-(J4-Pad1)
- J4 pad 7: Net-(J4-Pad7) -> Net-(J2-Pad2)
- J5 pad 2: Net-(J1-Pad1) -> Net-(J4-Pad2)
- J5 pad 3: Net-(J5-Pad3) -> Net-(J1-Pad1)
- J5 pad 5: Net-(J5-Pad5) -> Net-(J4-Pad1)
- J5 pad 6: Net-(J4-Pad2) -> Net-(J5-Pad6)
Routing:
- net Net-(J2-Pad2): track 0.00 -> 52.6 mm, vias 0 -> 1
- net Net-(J2-Pad6): track 39.2 -> 0.00 mm, vias 1 -> 0
- net Net-(J4-Pad1): track 0.00 -> 37.5 mm, vias 0 -> 1
- net Net-(J1-Pad2): track 0.00 -> 36.8 mm, vias 0 -> 1
- net Net-(J4-Pad2): track 66.5 -> 42.7 mm
- net Net-(J1-Pad3): track 99.2 -> 121.4 mm, vias 5 -> 1
- net Net-(J1-Pad1): track 56.4 -> 53.2 mm
- net Net-(J3-Pad6): track 29.7 -> 31.9 mm
- net Net-(J3-Pad5): track 26.1 -> 27.4 mm
- removed copper zone on B.Cu, net Net-(J1-Pad3)
- removed copper zone on F.Cu, net Net-(J1-Pad3)
Other:
- net class Default: trace_width 0.35 -> 0.4; via_dia 1.2 -> 1.5; via_drill 0.79375 -> 0.8

Commit message: shield
Routing:
- net Net-(J2-Pad2): track 52.6 -> 51.2 mm
Other:
- net class Default: via_dia 1.5 -> 1.6; via_drill 0.8 -> 0.9
Changed lines of the file:
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@@
     (links 13)
     (no_connects 1)
-    (area 116.510999 104.826999 166.699001 143.331001)
+    (area 116.246999 104.553 166.699001 143.884561)
     (thickness 1.6)
     (drawings 4)
-    (tracks 72)
+    (tracks 74)
     (zones 0)
     (modules 6)
@@
     (segment_width 0.2)
     (edge_width 0.15)
-    (via_size 1.5)
-    (via_drill 0.8)
+    (via_size 1.6)
+    (via_drill 0.9)
     (via_min_size 0.4)
     (via_min_drill 0.3)
@@
     (visible_elements 7FFFFFFF)
     (pcbplotparams
-      (layerselection 0x00000_80000001)
+      (layerselection 0x01000_80000001)
       (usegerberextensions false)
       (excludeedgelayer true)
@@
     (clearance 0.8)
     (trace_width 0.4)
-    (via_dia 1.5)
-    (via_drill 0.8)
+    (via_dia 1.6)
+    (via_drill 0.9)
     (uvia_dia 0.3)
     (uvia_drill 0.1)
@@
   (gr_line (start 166.624 143.256) (end 116.586 143.256) (angle 90) (layer Edge.Cuts) (width 0.15))
   (segment (start 132.588 117.602) (end 144.526 117.602) (width 0.4) (layer B.Cu) (net 1))
-  (segment (start 144.526 117.602) (end 148.59 113.538) (width 0.4) (layer B.Cu) (net 1) (status 800000))
+  (segment (start 144.526 117.602) (end 148.59 113.538) (width 0.4) (layer B.Cu) (net 1))
   (segment (start 132.588 123.444) (end 132.588 117.602) (width 0.4) (layer B.Cu) (net 1))
   (segment (start 132.588 117.602) (end 132.588 113.792) (width 0.4) (layer B.Cu) (net 1))
@@
   (segment (start 132.588 133.858) (end 132.588 123.444) (width 0.4) (layer B.Cu) (net 1))
   (segment (start 129.286 137.16) (end 132.588 133.858) (width 0.4) (layer B.Cu) (net 1))
-  (via (at 129.286 137.16) (size 1.5) (drill 0.8) (layers F.Cu B.Cu) (net 1))
-  (segment (start 132.842 110.998) (end 128.27 110.998) (width 0.4) (layer B.Cu) (net 2) (status 400000))
-  (segment (start 127 134.62) (end 118.872 134.62) (width 0.4) (layer F.Cu) (net 2) (status 800000))
-  (via (at 127 134.62) (size 1.5) (drill 0.8) (layers F.Cu B.Cu) (net 2))
+  (via (at 129.286 137.16) (size 1.6) (drill 0.9) (layers F.Cu B.Cu) (net 1))
+  (segment (start 132.842 110.998) (end 128.27 110.998) (width 0.4) (layer B.Cu) (net 2))
+  (segment (start 127 134.62) (end 118.872 134.62) (width 0.4) (layer F.Cu) (net 2))
+  (via (at 127 134.62) (size 1.6) (drill 0.9) (layers F.Cu B.Cu) (net 2))
   (segment (start 127 112.268) (end 127 134.62) (width 0.4) (layer B.Cu) (net 2))
   (segment (start 128.27 110.998) (end 127 112.268) (width 0.4) (layer B.Cu) (net 2))
   (segment (start 135.128 132.08) (end 135.128 134.366) (width 0.4) (layer B.Cu) (net 3))
-  (segment (start 140.716 113.538) (end 135.382 113.538) (width 0.4) (layer B.Cu) (net 3) (status 800000))
+  (segment (start 140.716 113.538) (end 135.382 113.538) (width 0.4) (layer B.Cu) (net 3))
   (segment (start 143.256 110.998) (end 140.716 113.538) (width 0.4) (layer B.Cu) (net 3))
   (segment (start 143.256 108.712) (end 143.256 110.998) (width 0.4) (layer B.Cu) (net 3))
@@
   (segment (start 130.048 139.446) (end 128.524 139.446) (width 0.4) (layer B.Cu) (net 3))
   (segment (start 135.128 134.366) (end 130.048 139.446) (width 0.4) (layer B.Cu) (net 3))
-  (segment (start 151.13 113.538) (end 151.13 116.078) (width 0.4) (layer B.Cu) (net 3) (status 400000))
+  (segment (start 151.13 113.538) (end 151.13 116.078) (width 0.4) (layer B.Cu) (net 3))
   (segment (start 147.32 119.888) (end 135.128 119.888) (width 0.4) (layer B.Cu) (net 3))
   (segment (start 151.13 116.078) (end 147.32 119.888) (width 0.4) (layer B.Cu) (net 3))
@@
   (segment (start 118.872 132.08) (end 135.128 132.08) (width 0.4) (layer F.Cu) (net 3))
   (segment (start 135.128 132.08) (end 135.128 123.444) (width 0.4) (layer B.Cu) (net 3))
-  (via (at 135.128 132.08) (size 1.5) (drill 0.8) (layers F.Cu B.Cu) (net 3))
-  (segment (start 164.02304 128.8796) (end 160.6296 128.8796) (width 0.4) (layer F.Cu) (net 16) (status 400000))
-  (segment (start 140.208 125.73) (end 140.208 123.444) (width 0.4) (layer B.Cu) (net 16) (status 800000))
+  (via (at 135.128 132.08) (size 1.6) (drill 0.9) (layers F.Cu B.Cu) (net 3))
+  (segment (start 164.02304 128.8796) (end 160.6296 128.8796) (width 0.4) (layer F.Cu) (net 16))
+  (segment (start 140.208 125.73) (end 140.208 123.444) (width 0.4) (layer B.Cu) (net 16))
   (segment (start 143.256 128.778) (end 140.208 125.73) (width 0.4) (layer B.Cu) (net 16))
   (segment (start 160.528 128.778) (end 143.256 128.778) (width 0.4) (layer B.Cu) (net 16))
-  (via (at 160.528 128.778) (size 1.5) (drill 0.8) (layers F.Cu B.Cu) (net 16))
+  (via (at 160.528 128.778) (size 1.6) (drill 0.9) (layers F.Cu B.Cu) (net 16))
   (segment (start 160.6296 128.8796) (end 160.528 128.778) (width 0.4) (layer F.Cu) (net 16))
-  (segment (start 164.02304 131.4196) (end 159.3596 131.4196) (width 0.4) (layer F.Cu) (net 17) (status 400000))
-  (segment (start 137.668 127.254) (end 137.668 123.444) (width 0.4) (layer B.Cu) (net 17) (status 800000))
+  (segment (start 164.02304 131.4196) (end 159.3596 131.4196) (width 0.4) (layer F.Cu) (net 17))
+  (segment (start 137.668 127.254) (end 137.668 123.444) (width 0.4) (layer B.Cu) (net 17))
   (segment (start 141.478 131.064) (end 137.668 127.254) (width 0.4) (layer B.Cu) (net 17))
   (segment (start 159.004 131.064) (end 141.478 131.064) (width 0.4) (layer B.Cu) (net 17))
-  (via (at 159.004 131.064) (size 1.5) (drill 0.8) (layers F.Cu B.Cu) (net 17))
+  (via (at 159.004 131.064) (size 1.6) (drill 0.9) (layers F.Cu B.Cu) (net 17))
   (segment (start 159.3596 131.4196) (end 159.004 131.064) (width 0.4) (layer F.Cu) (net 17))
-  (segment (start 148.59 110.998) (end 146.05 110.998) (width 0.4) (layer B.Cu) (net 18) (status 400000))
-  (segment (start 156.62656 136.56056) (end 156.62656 141.25956) (width 0.4) (layer F.Cu) (net 18) (status 800000))
+  (segment (start 148.59 110.998) (end 146.05 110.998) (width 0.4) (layer B.Cu) (net 18))
+  (segment (start 156.62656 136.56056) (end 156.62656 141.25956) (width 0.4) (layer F.Cu) (net 18))
   (segment (start 154.686 134.62) (end 156.62656 136.56056) (width 0.4) (layer F.Cu) (net 18))
   (segment (start 154.686 118.872) (end 154.686 134.62) (width 0.4) (layer F.Cu) (net 18))
@@
   (segment (start 146.558 116.586) (end 152.4 116.586) (width 0.4) (layer F.Cu) (net 18))
   (segment (start 143.51 113.538) (end 146.558 116.586) (width 0.4) (layer F.Cu) (net 18))
-  (via (at 143.51 113.538) (size 1.5) (drill 0.8) (layers F.Cu B.Cu) (net 18))
+  (via (at 143.51 113.538) (size 1.6) (drill 0.9) (layers F.Cu B.Cu) (net 18))
   (segment (start 146.05 110.998) (end 143.51 113.538) (width 0.4) (layer B.Cu) (net 18))
-  (segment (start 135.382 110.998) (end 140.716 110.998) (width 0.4) (layer B.Cu) (net 27) (status 400000))
-  (segment (start 143.92656 135.21944) (end 143.92656 141.25956) (width 0.4) (layer F.Cu) (net 27) (status 800000))
+  (segment (start 139.7 110.998) (end 140.081 110.998) (width 0.4) (layer B.Cu) (net 27))
+  (segment (start 141.224 112.395) (end 141.224 115.824) (width 0.4) (layer F.Cu) (net 27))
+  (segment (start 141.224 115.824) (end 144.272 118.872) (width 0.4) (layer F.Cu) (net 27))
+  (segment (start 144.272 118.872) (end 151.892 118.872) (width 0.4) (layer F.Cu) (net 27))
+  (segment (start 151.892 118.872) (end 153.162 120.142) (width 0.4) (layer F.Cu) (net 27))
+  (segment (start 153.162 120.142) (end 153.162 130.302) (width 0.4) (layer F.Cu) (net 27))
+  (segment (start 153.162 130.302) (end 149.86 133.604) (width 0.4) (layer F.Cu) (net 27))
+  (segment (start 149.86 133.604) (end 145.542 133.604) (width 0.4) (layer F.Cu) (net 27))
   (segment (start 145.542 133.604) (end 143.92656 135.21944) (width 0.4) (layer F.Cu) (net 27))
-  (segment (start 149.86 133.604) (end 145.542 133.604) (width 0.4) (layer F.Cu) (net 27))
-  (segment (start 153.162 130.302) (end 149.86 133.604) (width 0.4) (layer F.Cu) (net 27))
-  (segment (start 153.162 120.142) (end 153.162 130.302) (width 0.4) (layer F.Cu) (net 27))
-  (segment (start 151.892 118.872) (end 153.162 120.142) (width 0.4) (layer F.Cu) (net 27))
-  (segment (start 144.272 118.872) (end 151.892 118.872) (width 0.4) (layer F.Cu) (net 27))
-  (segment (start 141.224 115.824) (end 144.272 118.872) (width 0.4) (layer F.Cu) (net 27))
-  (segment (start 141.224 110.49) (end 141.224 115.824) (width 0.4) (layer F.Cu) (net 27))
-  (via (at 141.224 110.49) (size 1.5) (drill 0.8) (layers F.Cu B.Cu) (net 27))
-  (segment (start 140.716 110.998) (end 141.224 110.49) (width 0.4) (layer B.Cu) (net 27))
-  (segment (start 151.13 110.998) (end 155.702 110.998) (width 0.4) (layer B.Cu) (net 28) (status 400000))
-  (segment (start 159.16656 136.30656) (end 159.16656 141.25956) (width 0.4) (layer F.Cu) (net 28) (status 800000))
+  (segment (start 143.92656 141.25956) (end 143.92656 135.21944) (width 0.4) (layer F.Cu) (net 27))
+  (segment (start 139.7 110.998) (end 135.382 110.998) (width 0.4) (layer B.Cu) (net 27) (status 800000))
+  (segment (start 141.224 112.141) (end 141.224 112.395) (width 0.4) (layer F.Cu) (net 27))
+  (segment (start 140.081 110.998) (end 141.224 112.141) (width 0.4) (layer F.Cu) (net 27))
+  (via (at 140.081 110.998) (size 1.6) (drill 0.9) (layers F.Cu B.Cu) (net 27))
+  (segment (start 151.13 110.998) (end 155.702 110.998) (width 0.4) (layer B.Cu) (net 28))
+  (segment (start 159.16656 136.30656) (end 159.16656 141.25956) (width 0.4) (layer F.Cu) (net 28))
   (segment (start 156.21 133.35) (end 159.16656 136.30656) (width 0.4) (layer F.Cu) (net 28))
   (segment (start 156.21 114.554) (end 156.21 133.35) (width 0.4) (layer F.Cu) (net 28))
   (segment (start 157.734 113.03) (end 156.21 114.554) (width 0.4) (layer F.Cu) (net 28))
-  (via (at 157.734 113.03) (size 1.5) (drill 0.8) (layers F.Cu B.Cu) (net 28))
+  (via (at 157.734 113.03) (size 1.6) (drill 0.9) (layers F.Cu B.Cu) (net 28))
   (segment (start 155.702 110.998) (end 157.734 113.03) (width 0.4) (layer B.Cu) (net 28))
 )
